File: Nixie Tube Clock/Nixie Tube Clock.sch (KiCad schematic (older format))
At the start: 9 parts

Commit message: Finished the clock
Parts:
- added H1, H3, H4: MountingHole, MountingHole:MountingHole_3.2mm_M3_Pad_Via, symbol Mechanical:MountingHole
- added J3, J4: Conn_01x02, TerminalBlock:TerminalBlock_Altech_AK300-2_P5.00mm, symbol Connector_Generic:Conn_01x02
- added J5: Conn_02x04_Counter_Clockwise, Connector_PinHeader_2.54mm:PinHeader_2x04_P2.54mm_Vertical, symbol Connector_Generic:Conn_02x04_Counter_Clockwise
- added JP1: Jumper, Connector_PinHeader_2.54mm:PinHeader_2x01_P2.54mm_Vertical, symbol Device:Jumper
- added JP2: Jumper, Connector_PinHeader_2.54mm:PinHeader_1x02_P2.54mm_Vertical, symbol Device:Jumper
- added R2: 1K, Resistor_THT:R_Axial_DIN0207_L6.3mm_D2.5mm_P10.16mm_Horizontal, symbol Device:R_Small
- added R3: 2.2K, Resistor_THT:R_Axial_DIN0207_L6.3mm_D2.5mm_P10.16mm_Horizontal, symbol Device:R_Small
- added R8: 10K, Resistor_THT:R_Axial_DIN0207_L6.3mm_D2.5mm_P10.16mm_Horizontal, symbol Device:R_Small
- added SW1: SW_Push, Button_Switch_THT:SW_PUSH_6mm, symbol Switch:SW_Push
- added TP1: ~RST, TestPoint:TestPoint_Pad_2.0x2.0mm, symbol Connector:TestPoint
- added TP2: +12V, TestPoint:TestPoint_Pad_2.0x2.0mm, symbol Connector:TestPoint
- added TP3: +170V, TestPoint:TestPoint_Pad_2.0x2.0mm, symbol Connector:TestPoint
- added TP4: GND, TestPoint:TestPoint_Pad_2.0x2.0mm, symbol Connector:TestPoint
- added TP5: +5V, TestPoint:TestPoint_Pad_2.0x2.0mm, symbol Connector:TestPoint
- added TP6: ESP_RST, TestPoint:TestPoint_Pad_2.0x2.0mm, symbol Connector:TestPoint
- added TP7: +3V3, TestPoint:TestPoint_Pad_2.0x2.0mm, symbol Connector:TestPoint
- added U2: uA7805, Package_TO_SOT_THT:TO-220-3_Vertical, symbol Regulator_Linear:uA7805
- added U3: LM1084-3.3, Package_TO_SOT_THT:TO-220-3_Vertical, symbol Regulator_Linear:LM1084-3.3
- C1, C2, C3, C4: renamed from C?; footprint (none) -> Capacitor_THT:CP_Radial_D4.0mm_P2.00mm
- J1, J2: renamed from J?; footprint (none) -> Connector_PinHeader_2.54mm:PinHeader_1x06_P2.54mm_Vertical
- R1: renamed from R?; footprint (none) -> Resistor_THT:R_Axial_DIN0207_L6.3mm_D2.5mm_P10.16mm_Horizontal
- Y1: renamed from Y?; footprint (none) -> Crystal:Crystal_HC49-U_Vertical
- gave numbers to parts that had none: 1
Connections:
- net +5V: now also TP5.1, U2.3 (OUT)
- net GND: now also J3.2 (Pin_2), J4.2 (Pin_2), J5.1 (Pin_1), R3.1, SW1.2, TP4.1, U2.2 (GND), U3.1 (GND)
- net RX: now also JP2.2
- net TX: now also R2.2
- net ~RST: now also SW1.1, TP1.1
- net ESP_RST: now reaches U1.4 (PD2)
- net ESP_RST: now also J5.6 (Pin_6), TP6.1
- new net: J5.2 (Pin_2), JP1.2
- new net: J5.7 (Pin_7), JP2.1
- new net: JP1.1, R2.1, R3.2
- new net +12V: J3.1 (Pin_1), TP2.1, U2.1 (IN), U3.3 (VI)
- new net +170V: J4.1 (Pin_1), TP3.1
- new net +3V3: J5.8 (Pin_8), R8.2, TP7.1, U3.2 (VO)
- new net CH_EN: J5.4 (Pin_4), R8.1
- new net ESP_GPIO0: J5.5 (Pin_5)
- new net ESP_GPIO2: J5.3 (Pin_3)
Other:
- moved on the sheet: J1, J2
